Commit message: gen_urdf.sh: build mtu32_description from colcon_ws/src (the robots' source)
The sim's URDFs were generated from a separate copy of mtu32_husky in
sim/colcon_ws, frozen on 2026-09-28. The robots (and the real ones) use
colcon_ws/src/mtu32_husky, whose robot_description.urdf.xacro has since moved
to sensor_arch_v2 (tall arch, GNSS domes on top), dropped the e-stop/button
links and added the D405 camera_1 on the arm. a300_00036 in Isaac therefore
showed the old low arch with floating GNSS domes while Foxglove showed the
right model.

gen_urdf.sh now mounts colcon_ws/src/mtu32_husky/mtu32_description read-only
and builds it in the throwaway container's /tmp. Regenerated: a300_00036 and
a300_00037 (the Jackals' xacro was unchanged); the meshes they no longer use
are removed. a300_00036 now also gets the wrist camera (derived wrist_camera),
which costs ~13% fps with one robot (19 -> 16). Drive test and camera_1
topics checked live.

Co-Authored-By: Claude Opus 5.5 <noreply@anthropic.com>

File: sim/assets/a300_00036/a300_00036.urdf (robot description, URDF)
Before this commit: robot a300_00036, 109 links, 108 joints
Links:
- removed link button_link
- removed link estop_link
- added link camera_1_bottom_screw_frame
- added link camera_1_link, mass 0.072; collision box size=0.023 0.042 0.042; visual mesh filename=meshes/realsense2_description/meshes/d405.stl scale=0.001 0.001 0.001
- link arch_link: geometry collision box size=0.17 0.05 0.145; visual mesh filename=meshes/mtu32_description/meshes/sensor_arch_v2.STL
Joints:
- removed joint button_joint
- removed joint estop_joint
- added joint camera_1_joint: type fixed, parent arm_0_end_effector_link, child camera_1_bottom_screw_frame, origin xyz=0.045 0.0 0.0 rpy=0.0 0.0 0.0
- added joint camera_1_link_joint: type fixed, parent camera_1_bottom_screw_frame, child camera_1_link, origin xyz=0.01085 0.009 0.021 rpy=0 0 0

File: sim/assets/a300_00037/a300_00037.urdf (robot description, URDF)
Before this commit: robot a300_00037, 118 links, 117 joints
Links:
- removed link button_link
- removed link estop_link
- link arch_link: geometry collision box size=0.17 0.05 0.145; visual mesh filename=meshes/mtu32_description/meshes/sensor_arch_v2.STL
Joints:
- removed joint button_joint
- removed joint estop_joint

Commit message: sim/assets: regenerate with clearpath 2.9.17 and zenoh robot.yamls
robot.yaml copies follow robot_data's rmw_zenoh_cpp. a300_00036/00037:
2.9.17 gives the Hokuyo UST a collision box, so lidar2d_0_link (and the
wireless charger's face/lidar mount frames) are no longer merged into
wireless_charger_link. Drive test and lidar scan (no self-hits) checked.

Co-Authored-By: Claude Opus 5.5 <noreply@anthropic.com>

File: sim/assets/a300_00036/a300_00036.urdf (robot description, URDF)
Before this commit: robot a300_00036, 109 links, 108 joints
Links:
- added link lidar2d_0_link; collision box size=0.06 0.06 0.08; visual mesh filename=meshes/clearpath_sensors_description/meshes/hokuyo_ust.stl
- added link wireless_charger_face
- added link wireless_charger_lidar_mount
- link wireless_charger_link: geometry collision box size=0.170 0.145 0.195; visual mesh filename=meshes/clearpath_platform_description/meshes/a300/attachmen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 scale=0.001 0.001 0.001
Joints:
- added joint lidar2d_0_joint: type fixed, parent wireless_charger_lidar_mount, child lidar2d_0_link, origin xyz=0.0 0.0 0.0 rpy=0.0 0.0 0.0
- added joint wireless_charger_face_joint: type fixed, parent wireless_charger_link, child wireless_charger_face, origin xyz=0 -0.34 0.15 rpy=0 0 -1.5707963267948966
- added joint wireless_charger_lidar_link: type fixed, parent wireless_charger_face, child wireless_charger_lidar_mount, origin xyz=-0.065 0 0.125 rpy=0 0 0
- joint charger_0_joint: origin xyz=-1.8369702e-19 -0.337 0.16 rpy=3.14159265 2.65358979e-06 1.57079633 -> xyz=-0.003 0.0 0.01 rpy=0.0 3.14159 0.0; parent wireless_charger_link -> wireless_charger_face
- joint lidar2d_0_laser_joint: origin xyz=-3.9801021e-18 -0.275 0.3224 rpy=0 -0 -1.57079633 -> xyz=0 0 0.0474 rpy=0 0 0; parent wireless_charger_link -> lidar2d_0_link

File: sim/assets/a300_00037/a300_00037.urdf (robot description, URDF)
Before this commit: robot a300_00037, 116 links, 115 joints
Links:
- added link lidar2d_0_link; collision box size=0.06 0.06 0.08; visual mesh filename=meshes/clearpath_sensors_description/meshes/hokuyo_ust.stl
- added link wireless_charger_face
- added link wireless_charger_lidar_mount
- link wireless_charger_link: geometry collision box size=0.170 0.145 0.195; visual mesh filename=meshes/clearpath_platform_description/meshes/a300/attachmen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 scale=0.001 0.001 0.001
Joints:
- added joint lidar2d_0_joint: type fixed, parent wireless_charger_lidar_mount, child lidar2d_0_link, origin xyz=0.0 0.0 0.0 rpy=0.0 0.0 0.0
- added joint wireless_charger_face_joint: type fixed, parent wireless_charger_link, child wireless_charger_face, origin xyz=0 -0.34 0.15 rpy=0 0 -1.5707963267948966
- added joint wireless_charger_lidar_link: type fixed, parent wireless_charger_face, child wireless_charger_lidar_mount, origin xyz=-0.065 0 0.125 rpy=0 0 0
- joint charger_0_joint: origin xyz=-1.8369702e-19 -0.337 0.16 rpy=3.14159265 2.65358979e-06 1.57079633 -> xyz=-0.003 0.0 0.01 rpy=0.0 3.14159 0.0; parent wireless_charger_link -> wireless_charger_face
- joint lidar2d_0_laser_joint: origin xyz=-3.9801021e-18 -0.275 0.3224 rpy=0 -0 -1.57079633 -> xyz=0 0 0.0474 rpy=0 0 0; parent wireless_charger_link -> lidar2d_0_link
